Commit message: Add files via upload

File: turtlebot3_simulations/turtlebot3_gazebo/urdf/turtlebot3_burger.urdf (robot description, URDF)
Before this commit: robot turtlebot3_burger, 8 links, 7 joints
Links:
- link velodyne_link: geometry collision cylinder length=0.2 radius=0.04; visual cylinder length=0.2 radius=0.04
Joints:
- joint velodyne_joint: origin xyz=0 0 0.25 rpy=0 0 0 -> xyz=10 0.1 0.25 rpy=0 0 0
